Commit message: updated urdf to include camera

File: tank_ws/src/tankbot/urdf/tankbot.urdf (robot description, URDF)
Before this commit: robot tankbot, 21 links, 20 joints
Links:
- added link lidar_front_imu, mass 0.01
- added link lidar_rear_imu, mass 0.01
Joints:
- added joint lidar_front_to_imu: type fixed, parent lidar_front, child lidar_front_imu, origin xyz=0 0 0 rpy=0 0 0
- added joint lidar_rear_to_imu: type fixed, parent lidar_rear, child lidar_rear_imu, origin xyz=0 0 0 rpy=0 0 0
- joint base_to_gnss: origin xyz=0.0 0 0.25 rpy=0 0 0 -> xyz=0 0 0 rpy=0 0 0
