Commit message: with lidar

File: tank_ws/src/master_bot/urdf/master_bot.urdf (robot description, URDF)
Before this commit: robot master_bot, 17 links, 16 joints
Links:
- added link base_footprint; visual box size=0.001 0.001 0.001
Joints:
- added joint base_footprint_joint: type fixed, parent base_footprint, child base_link, origin xyz=0 0 0.5 rpy=0 0 0

Commit message: Swap l_FL2 and l_BL2 link names in URDF to match physical lidar positions
- Physical front mount (forward position) is now l_BL2
- Physical rear mount (backward position) is now l_FL2
- Updated Gazebo sensor references
- Updated pointcloud_frame_fixer to use swapped frame names
- This aligns URDF with actual lidar data from drivers

File: tank_ws/src/master_bot/urdf/master_bot.urdf (robot description, URDF)
Before this commit: robot master_bot, 18 links, 17 joints
Links:
- link l_BL2: mass 0.022313 -> 0.058407; geometry collision mesh filename=package://master_bot/meshes/l_FL2.STL; visual mesh filename=package://master_bot/meshes/l_FL2.STL
- link l_FL2: mass 0.058407 -> 0.022313; geometry collision mesh filename=package://master_bot/meshes/l_BL2.STL; visual mesh filename=package://master_bot/meshes/l_BL2.STL
Joints:
- joint j_BL2: origin xyz=0.32674 0 -0.17729 rpy=-3.1416 1.309 -3.1416 -> xyz=-0.26408 0 -0.17156 rpy=0 -1.5708 0
- joint j_FL2: origin xyz=-0.26408 0 -0.17156 rpy=0 -1.5708 0 -> xyz=0.32674 0 -0.17729 rpy=-3.1416 1.309 -3.1416

Commit message: Rotate both LiDAR links 180 degrees around Z-axis
- l_BL2 (front position): yaw 0 → 3.14159 (180°)
- l_FL2 (rear position): yaw -3.1416 → 0 (180° rotation)
- This corrects the physical orientation of the LiDAR sensors

File: tank_ws/src/master_bot/urdf/master_bot.urdf (robot description, URDF)
Before this commit: robot master_bot, 18 links, 17 joints
Joints:
- joint j_BL2: origin xyz=-0.26408 0 -0.17156 rpy=0 -1.5708 0 -> xyz=-0.26408 0 -0.17156 rpy=0 -1.5708 3.14159
- joint j_FL2: origin xyz=0.32674 0 -0.17729 rpy=-3.1416 1.309 -3.1416 -> xyz=0.32674 0 -0.17729 rpy=-3.1416 1.309 0

Commit message: Revert rotation changes - only swap link names, keep original orientations
- l_BL2 at forward position: xyz=(-0.26408 0 -0.17156) rpy=(0 -1.5708 0)
- l_FL2 at rear position: xyz=(0.32674 0 -0.17729) rpy=(-3.1416 1.309 -3.1416)
- Names are swapped but positions and orientations remain as originally designed

File: tank_ws/src/master_bot/urdf/master_bot.urdf (robot description, URDF)
Before this commit: robot master_bot, 18 links, 17 joints
Joints:
- joint j_BL2: origin xyz=-0.26408 0 -0.17156 rpy=0 -1.5708 3.14159 -> xyz=-0.26408 0 -0.17156 rpy=0 -1.5708 0
- joint j_FL2: origin xyz=0.32674 0 -0.17729 rpy=-3.1416 1.309 0 -> xyz=0.32674 0 -0.17729 rpy=-3.1416 1.309 -3.1416

Commit message: Rotate front lidar (l_BL2) 90° clockwise around Z-axis
- Changed rpy from (0 -1.5708 0) to (0 -1.5708 -1.5708)
- Yaw rotated -90° (clockwise) to correct lidar orientation

File: tank_ws/src/master_bot/urdf/master_bot.urdf (robot description, URDF)
Before this commit: robot master_bot, 18 links, 17 joints
Joints:
- joint j_BL2: origin xyz=-0.26408 0 -0.17156 rpy=0 -1.5708 0 -> xyz=-0.26408 0 -0.17156 rpy=0 -1.5708 -1.5708

Commit message: Revert front lidar rotation - back to original orientation
- Changed rpy back from (0 -1.5708 -1.5708) to (0 -1.5708 0)
- Front lidar (l_BL2) at original orientation

File: tank_ws/src/master_bot/urdf/master_bot.urdf (robot description, URDF)
Before this commit: robot master_bot, 18 links, 17 joints
Joints:
- joint j_BL2: origin xyz=-0.26408 0 -0.17156 rpy=0 -1.5708 -1.5708 -> xyz=-0.26408 0 -0.17156 rpy=0 -1.5708 0

Commit message: Add GNSS antenna link 10cm left of base_link
- Added gnss_link with orange cylinder visualization
- Fixed joint positioned at y=0.1 (10cm left of base_link)
- Mass: 0.05kg (ZED-F9P antenna)
- Cylinder dimensions: 2.5cm radius, 1cm height

File: tank_ws/src/master_bot/urdf/master_bot.urdf (robot description, URDF)
Before this commit: robot master_bot, 18 links, 17 joints
Links:
- added link gnss_link, mass 0.05; collision cylinder length=0.01 radius=0.025; visual cylinder length=0.01 radius=0.025
Joints:
- added joint gnss_joint: type fixed, parent base_link, child gnss_link, origin xyz=0 0.1 0 rpy=0 0 0
